File: hardware/open-TWIST_rev0/Power_supplies.kicad_sch (KiCad schematic)
At the start: 202 parts, among them J1 Jack-DC, SW1 SW_SPDT, U10 TPS7A4701RGWR, U11 LM73100RPWR, U12 L78L05_SOT89, U13 LMR14050SDDAQ1, U14 LTC6902, U2 ADP5071, U3 ADP5070, U4 ADP5070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

Commit message: work on readme
Connections:
- net SYNC_DC_5VD renamed SYNC_DC_3V3
Other:
- note added: "why????"
Changed lines of the file:
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@@
 		)
 	)
+	(text "why????"
+		(exclude_from_sim no)
+		(at 346.202 64.262 0)
+		(effects
+			(font
+				(size 2.54 2.54)
+			)
+			(justify left bottom)
+		)
+	)
 	(text "Fs = 2.2MHz"
 		(exclude_from_sim no)
@@
 		)
 	)
-	(global_label "SYNC_DC_5VD"
+	(global_label "SYNC_DC_3V3"
 		(shape output)
 		(at 381 151.13 0)
@@
 		)
 		(property "Intersheetrefs" "${INTERSHEET_REFS}"
-			(at 396.9271 151.13 0)
+			(at 396.8666 151.13 0)
 			(effects
 				(font
@@
 		)
 	)
-	(global_label "SYNC_DC_5VD"
+	(global_label "SYNC_DC_3V3"
 		(shape input)
 		(at 308.61 100.33 180)
@@
 		)
 		(property "Intersheetrefs" "${INTERSHEET_REFS}"
-			(at 292.6829 100.33 0)
+			(at 292.7434 100.33 0)
 			(effects
 				(font
