File: hardware/open-TWIST_rev0/USB.kicad_sch (KiCad schematic)
At the start: 118 parts, among them J2 UJ31-CH-G1-SMT-TR, P1 USB_C_Plug, U86 ECMF04-4HSWM10, U87 ECMF02-2AMX6, U88 FT601Q-B, U89 USB2422-I/MJ, U90 93LC46BT-I/OT, U91 FT2232HQ, Y1 30MHz 20ppm, Y2 24MHz 20ppm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

Commit message: work on readme
Connections:
- net FT601_BE0: no longer R252.2
- new net FT601_BE1: R252.2
Changed lines of the file:
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@@
 		)
 	)
-	(hierarchical_label "FT601_BE0"
+	(hierarchical_label "FT601_BE1"
 		(shape input)
 		(at 187.96 63.5 0)
