File: hardware/open-TWIST_rev0/open-TWIST_rev0.kicad_sch (KiCad schematic)
At the start: 10 parts, among them U1 REF35120QDBVR

Commit message: work on readme
Other:
- sheet USB ports: added FT601_BE1; removed none
Changed lines of the file:
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@@
 		)
 		(instances
-			(project "TWIST_V2"
+			(project "open-TWIST_rev0"
 				(path "/e33fddd6-be85-4cf9-a6aa-44cdd8b2669a"
 					(page "10")
@@
 			)
 		)
+		(pin "FT601_BE1" input
+			(at 80.01 215.9 180)
+			(effects
+				(font
+					(size 1.27 1.27)
+				)
+				(justify left)
+			)
+		)
 		(instances
-			(project "TWIST_V2"
+			(project "open-TWIST_rev0"
 				(path "/e33fddd6-be85-4cf9-a6aa-44cdd8b2669a"
 					(page "22")
@@
 		)
 		(instances
-			(project "TWIST_V2"
+			(project "open-TWIST_rev0"
 				(path "/e33fddd6-be85-4cf9-a6aa-44cdd8b2669a"
 					(page "23")
@@
 		)
 		(instances
-			(project "TWIST_V2"
+			(project "open-TWIST_rev0"
 				(path "/e33fddd6-be85-4cf9-a6aa-44cdd8b2669a"
 					(page "2")
@@
 		)
 		(instances
-			(project "TWIST_V2"
+			(project "open-TWIST_rev0"
 				(path "/e33fddd6-be85-4cf9-a6aa-44cdd8b2669a"
 					(page "24")
@@
 		)
 		(instances
-			(project "TWIST_V2"
+			(project "open-TWIST_rev0"
 				(path "/e33fddd6-be85-4cf9-a6aa-44cdd8b2669a"
 					(page "6")
@@
 		)
 		(instances
-			(project "TWIST_V2"
+			(project "open-TWIST_rev0"
 				(path "/e33fddd6-be85-4cf9-a6aa-44cdd8b2669a"
 					(page "3")
